Commit message: Added support for setting the wheel color. The mecanum robot now has silver wheels, and the skidsteer robot has black wheels.

File: urdf/smp.urdf.xacro (robot description, xacro)
@@ -125,6 +125,5 @@
                 </geometry>
                 <origin rpy="${yreflect*1.57075} ${xreflect*1.57075} 0" xyz="0 0 0"/>
-                <!--<material name="silver"/>-->
-		<material name="black" />
+		<material name="${wheelColor}" />
             </visual>
         </link>

File: urdf/smp_mecanum.urdf.xacro (robot description, xacro)
@@ -11,7 +11,5 @@
     <!--Distance between left and right wheels-->
     <property name="wheelTrack" value="0.5969"/>
-    <!--<property name="heightFromGround" value="0.202"/>-->
-    <!--<property name="heightFromGround" value="0.216"/>-->
-    <!--<property name="heightFromGround" value="0.26035"/>-->
+    <xacro:property name="wheelColor" value="silver"/>
     <smp_base/>
 </robot>

File: urdf/smp_skidsteer.urdf.xacro (robot description, xacro)
@@ -11,6 +11,5 @@
     <!--Distance between left and right wheels-->
     <property name="wheelTrack" value="0.5461"/>
-    <!--<property name="heightFromGround" value="0.202"/>-->
-    <!--<property name="heightFromGround" value="0.71755"/>-->
+    <xacro:property name="wheelColor" value="black"/>
     <smp_base/>
 </robot>

Commit message: Changed smp urdf file wheel joint names to match exist stuff.

File: urdf/smp.urdf.xacro (robot description, xacro)
@@ -128,5 +128,5 @@
             </visual>
         </link>
-        <joint name="${xfix}_${yfix}_shaft_to_${xfix}_${yfix}_wheel" type="continuous">
+        <joint name="${xfix}_${yfix}_wheel_joint" type="continuous">
             <parent link="${xfix}_${yfix}_shaft"/>
             <child link="${xfix}_${yfix}_wheel"/>
@@ -291,10 +291,10 @@
     <xacro:leg xfix="front" yfix="left" xreflect="1" yreflect="1" />
     <xacro:leg xfix="front" yfix="right" xreflect="1" yreflect="-1" />
-    <xacro:leg xfix="rear" yfix="left" xreflect="-1" yreflect="1" />
-    <xacro:leg xfix="rear" yfix="right" xreflect="-1" yreflect="-1" />
+    <xacro:leg xfix="back" yfix="left" xreflect="-1" yreflect="1" />
+    <xacro:leg xfix="back" yfix="right" xreflect="-1" yreflect="-1" />
     <xacro:wheel xfix="front" yfix="left" xreflect="1" yreflect="1" />
     <xacro:wheel xfix="front" yfix="right" xreflect="1" yreflect="-1" />
-    <xacro:wheel xfix="rear" yfix="left" xreflect="-1" yreflect="1" />
-    <xacro:wheel xfix="rear" yfix="right" xreflect="-1" yreflect="-1" />
+    <xacro:wheel xfix="back" yfix="left" xreflect="-1" yreflect="1" />
+    <xacro:wheel xfix="back" yfix="right" xreflect="-1" yreflect="-1" />
     </xacro:macro>
 </robot>

Commit message: Fixed wheel joint name.

File: urdf/smp.urdf.xacro (robot description, xacro)
@@ -128,5 +128,5 @@
             </visual>
         </link>
-        <joint name="${xfix}_${yfix}_wheel_joint" type="continuous">
+        <joint name="wheel_${xfix}_${yfix}_joint" type="continuous">
             <parent link="${xfix}_${yfix}_shaft"/>
             <child link="${xfix}_${yfix}_wheel"/>
